File: pcb.kicad_sch (KiCad schematic)
At the start: 3 parts

Commit message: schematic done
Parts:
- removed BT1: CR2032, Battery:BatteryHolder_Keystone_3034_1x20mm, symbol Device:Battery_Cell
- removed D1: LED, LED_SMD:LED_0805_2012Metric, symbol Device:LED
- removed R1: 1k, Resistor_SMD:R_0805_2012Metric, symbol Device:R
- added C10, C11, C12 (x3), C6 (x9), C8, C9 (x2): 100n, Capacitor_SMD:C_0402_1005Metric, symbol Device:C_Small
- added C11, C3: 1u, Capacitor_SMD:C_0603_1608Metric, symbol Device:C_Small
- added C12, C14: 1u, Capacitor_SMD:C_0402_1005Metric, symbol Device:C_Small
- added C4: 4u7, Capacitor_SMD:C_0603_1608Metric, symbol Device:C_Small
- added C5, C7: 30p, Capacitor_SMD:C_0402_1005Metric, symbol Device:C_Small
- added D1: Yellow, symbol Device:LED_Small
- added D2: Orange, symbol Device:LED_Small
- added D3: Red, symbol Device:LED_Small
- added D4, D5: SMBJ6.0CA, Diode_SMD:D_SMB, symbol Device:D_TVS
- added H1, H2: MountingHole, MountingHole:MountingHole_2.2mm_M2, symbol Mechanical:MountingHole
- added J1: Conn_ARM_SWD_TagConnect_TC2030-NL, Connector:Tag-Connect_TC2030-IDC-NL_2x03_P1.27mm_Vertical, symbol Connector:Conn_ARM_SWD_TagConnect_TC2030-NL
- added J2: Conn_ARM_JTAG_SWD_10, symbol Connector:Conn_ARM_JTAG_SWD_10
- added J3: JST B04B-PASK, symbol Connector_Generic:Conn_01x04
- added P1: USB_C_Plug, Expansion_Card:USB_C_Plug_Molex_105444, symbol Connector:USB_C_Plug
- added Q1, Q2: AO3400A, Package_TO_SOT_SMD:SOT-23, symbol Transistor_FET:AO3400A
- added Q3, Q4: AO3401A, Package_TO_SOT_SMD:SOT-23, symbol Transistor_FET:AO3401A
- added R1, R2: 5.1k, Resistor_SMD:R_0402_1005Metric, symbol Device:R_Small
- added R10, R8, R9: 330R, symbol Device:R_Small
- added R11, R12, R13, R14, R15, R16, R17, R19: 100R, symbol Device:R_Small
- added R18, R20, R22, R4, R6: 10k, symbol Device:R_Small
- added R21, R5: 4k7, symbol Device:R_Small
- added R3: 0R, symbol Device:R_Small
- added R6: 1k5, Resistor_SMD:R_0402_1005Metric, symbol Device:R_Small
- added SW1: SW_Push, Button_Switch_SMD:SW_Push_SPST_NO_Alps_SKRK, symbol Switch:SW_Push
- added TP1, TP2, TP3, TP4: TestPoint, TestPoint:TestPoint_Pad_1.5x1.5mm, symbol Connector:TestPoint
- added U1: WE-TVS-82400102, Package_TO_SOT_SMD:SOT-23-6, symbol Power_Protection:WE-TVS-82400102
- added U3: STM32F103C8T6, Package_QFP:LQFP-48_7x7mm_P0.5mm, symbol MCU_ST_STM32F1:STM32F103C8Tx
- added U3: NCP360SNT1G, TSOP5_3X1P5_ONS, symbol 2023-04-20_05-50-10:NCP360SNT1G
- added U4: MCP1825S, symbol Regulator_Linear:MCP1825S
- added U5, U6, U7, U8: 74LVC2T45DC, Package_SO:VSSOP-8_2.3x2mm_P0.5mm, symbol Logic_LevelTranslator:74LVC2T45DC
- added Y1: 8MHz, Crystal:Crystal_SMD_5032-2Pin_5.0x3.2mm, symbol Device:Crystal_Small
Connections:
- net GND: now also C10.2, C11.2, C11.2, C12.2, C12.2, C12.2, C12.2, C14.2, C3.2, C4.2, C5.2, C6.2, C6.2, C6.2, C6.2, C6.2, C6.2, C6.2, C6.2, C6.2, C7.2, C8.2, C9.2, C9.2, D1.1 (K), D2.1 (K), D3.1 (K), D4.1 (A1), D5.1 (A1), J1.5 (GND), J2.3 (GND), J2.5 (GND), J2.9 (GNDDetect), J3.4 (Pin_4), P1.A1 (GND), P1.A12 (GND), P1.B1 (GND), P1.B12 (GND), P1.S1 (SHIELD), Q1.2 (S), Q2.2 (S), R1.2, R2.2, R22.1, R6.1, SW1.1, TP1.1, TP2.1, TP3.1, TP4.1, U1.2, U3.2 (GND), U3.23 (VSS), U3.3 (*EN), U3.35 (VSS), U3.44 (BOOT0), U3.47 (VSS), U3.8 (VSSA), U4.2 (GND), U5.4 (GND), U6.4 (GND), U7.4 (GND), U7.5 (DIR), U8.4 (GND)
- new net: D2.2 (A), R9.2
- new net: C9.1, R3.2, U3.7 (NRST)
- new net: D3.2 (A), R10.2
- new net: P1.A5 (CC), R1.1
- new net: P1.B5 (VCONN), R2.1
- new net: Q3.2 (S), Q4.2 (S), R20.2
- new net: D1.2 (A), R8.2
- new net: R4.1, SW1.2, U3.25 (PB12)
- new net +3V3: C10.1, C11.1, C12.1, C3.1, C4.1, C6.1, C6.1, C6.1, C6.1, C6.1, C8.1, C9.1, J1.1 (VCC), Q3.3 (D), R4.2, U3.1 (VBAT), U3.24 (VDD), U3.36 (VDD), U3.48 (VDD), U3.9 (VDDA), U4.3 (VO), U5.1 (VCCA), U5.5 (DIR), U6.1 (VCCA), U6.5 (DIR), U7.1 (VCCA), U8.1 (VCCA)
- new net HSE_IN: C7.1, U3.6 (PD1), Y1.2
- new net HSE_OUT: C5.1, U3.5 (PD0), Y1.1
- new net LED0: R8.1, U3.20 (PB2)
- new net LED1: R9.1, U3.21 (PB10)
- new net LED2: R10.1, U3.22 (PB11)
- new net PWR_BR: Q3.1 (G), Q4.1 (G), R20.1, U3.19 (PB1)
- new net RST: J2.10 (~{RESET}), R11.2
- new net RST_SENSE: Q2.3 (D), U3.17 (PA7)
- new net RXD: J3.3 (Pin_3), R17.2
- new net SSD+: P1.A6 (D+), U1.3
- new net SSD-: P1.A7 (D-), U1.1
- new net SWCLK: J1.4 (SWCLK), U3.37 (PA14)
- new net SWDIO: J1.2 (SWDIO), U3.34 (PA13)
- new net SWO: J1.6 (SWO), U3.39 (PB3)
- new net TCK: J2.4 (SWDCLK/TCK), R12.2
- new net TDI: J2.8 (NC/TDI), R15.2
- new net TDO: J2.6 (SWO/TDO), R14.2
- new net TMS: J2.2 (SWDIO/TMS), R13.2
- new net TMS_DIR: U3.11 (PA1), U8.5 (DIR)
- new net TPWR: D5.2 (A2), J2.1 (VTref), J3.1 (Pin_1), Q4.3 (D), R19.2, R21.2
- new net TPWR_MEAS: C12.1, R21.1, R22.2, U3.18 (PB0)
- new net TXD: J3.2 (Pin_2), R16.2
- new net USB_D+: R6.2, U1.4, U3.33 (PA12)
- new net USB_D-: U1.6, U3.32 (PA11)
- new net USB_PU: R6.1, U3.29 (PA8)
- new net VBUS: C14.1, R5.2, U3.5 (OUT), U4.1 (VI)
- new net VBUS_IN: C11.1, C12.1, P1.A4 (VBUS), P1.A9 (VBUS), P1.B4 (VBUS), P1.B9 (VBUS), U1.5, U3.1 (IN)
- new net VBUS_MEAS: C12.1, R5.1, R6.2, U3.38 (PA15)
- new net iRST: Q1.1 (G), U3.12 (PA2)
- new net iRXD: U3.31 (PA10), U7.3 (2A)
- new net iTCK: U3.15 (PA5), U6.2 (1A)
- new net iTDI: U3.13 (PA3), U6.3 (2A)
- new net iTDO: U3.16 (PA6), U3.43 (PB7), U7.2 (1A)
- new net iTMS: U3.14 (PA4), U8.3 (2A)
- new net iTXD: U3.30 (PA9), U5.3 (2A)
- new net nRST: J1.3 (~{RESET}), R3.1
- new net xRST: D4.2 (A2), Q1.3 (D), Q2.1 (G), R11.1, R18.2
- new net xRXD: R17.1, U7.6 (2B)
- new net xTCK: R12.1, U6.7 (1B)
- new net xTDI: R15.1, U6.6 (2B)
- new net xTDO: R14.1, U7.7 (1B)
- new net xTMS: R13.1, U8.6 (2B)
- new net xTPWR: C6.1, C6.1, C6.1, C6.1, R18.1, R19.1, U5.8 (VCCB), U6.8 (VCCB), U7.8 (VCCB), U8.8 (VCCB)
- new net xTXD: R16.1, U5.6 (2B)
- no-connect marks 0 -> 27
Other:
- note added: "-> <-"
- note added: "3V3 regulator stable with 1uF output cap."
- note added: "4.7u bulk decoupling + 100nF per VDD pin + 1u on VDDA"
- note added: "CL = 2 * (Cload - Cstray)"
- note added: "JTAG header mounted on side of board with 1/2 of pins on top and 1/2 on bottom"
- note added: "Level conversion & Target Frontend"
- note added: "Programming/debug header. Place in an accessible location close to the mcu."
- note added: "STM32F1 Microcontroller"
- note added: "STM32F103 requires external 1k5 pull-up on USB D+ line."
- note added: "Status LEDs"
- note added: "Tag Connect"
- note added: "UART header mounted sideways sticking off edge of board"
- note added: "USB and Regulator"

Commit message: Shrinking
Parts:
- removed C12: 1u, Capacitor_SMD:C_0402_1005Metric, symbol Device:C_Small
- removed D4, D5: SMBJ6.0CA, Diode_SMD:D_SMB, symbol Device:D_TVS
- removed R11, R12, R13, R14, R15, R16, R17, R19: 100R, symbol Device:R_Small
- removed U3: NCP360SNT1G, TSOP5_3X1P5_ONS, symbol 2023-04-20_05-50-10:NCP360SNT1G
- removed U4: MCP1825S, symbol Regulator_Linear:MCP1825S
- added RN1, RN2: 100R, symbol Device:R_Pack04_Split
- added U9: AP2112K-3.3, Package_TO_SOT_SMD:SOT-23-5, symbol Regulator_Linear:AP2112K-3.3
- C11, C3: footprint Capacitor_SMD:C_0603_1608Metric -> Capacitor_SMD:C_0402_1005Metric
- D1, D2, D3: footprint (none) -> Connectors:LED_THT_Edge Mount
- J2: footprint (none) -> Connectors:Cortex-10pin-sidemount
- J3: footprint (none) -> Connectors:JST B04B-PASK Edge Mount
- R10, R18, R20, R21, R22, R3, R4, R5, R6, R8, R9: footprint (none) -> Resistor_SMD:R_0402_1005Metric
Connections:
- net VBUS_IN is gone; now on net VBUS: C11.1, P1.A4 (VBUS), P1.A9 (VBUS), P1.B4 (VBUS), P1.B9 (VBUS), U1.5
- net +3V3: now also U9.5 (VOUT)
- net GND: now also U9.2 (GND)
- net RST: now also RN2.1 (R1.1)
- net RXD: now also RN2.3 (R3.1)
- net TCK: now also RN1.2 (R2.1)
- net TDI: now also RN1.4 (R4.1)
- net TDO: now also RN1.3 (R3.1)
- net TMS: now also RN1.1 (R1.1)
- net TPWR: now also RN2.4 (R4.1)
- net TXD: now also RN2.2 (R2.1)
- net VBUS: now also U9.1 (VIN), U9.3 (EN)
- net xRXD: now also RN2.6 (R3.2)
- net xTCK: now also RN1.7 (R2.2)
- net xTDI: now also RN1.5 (R4.2)
- net xTDO: now also RN1.6 (R3.2)
- net xTMS: now also RN1.8 (R1.2)
- net xTPWR: now also RN2.5 (R4.2)
- net xTXD: now also RN2.7 (R2.2)
- no-connect marks 27 -> 26
Other:
- note added: "3V3 regulator stable with 1uF ceramic output cap."
- note removed: "3V3 regulator stable with 1uF output cap."
- moved on the sheet: C14, C3

Commit message: Layout and routing
Parts:
- removed C6 (x2): 100n, Capacitor_SMD:C_0402_1005Metric, symbol Device:C_Small
- removed D1: Yellow, Connectors:LED_THT_Edge Mount, symbol Device:LED_Small
- removed J1: Conn_ARM_SWD_TagConnect_TC2030-NL, Connector:Tag-Connect_TC2030-IDC-NL_2x03_P1.27mm_Vertical, symbol Connector:Conn_ARM_SWD_TagConnect_TC2030-NL
- removed J3: JST B04B-PASK, Connectors:JST B04B-PASK Edge Mount, symbol Connector_Generic:Conn_01x04
- removed Q1, Q2: AO3400A, Package_TO_SOT_SMD:SOT-23, symbol Transistor_FET:AO3400A
- removed Q3, Q4: AO3401A, Package_TO_SOT_SMD:SOT-23, symbol Transistor_FET:AO3401A
- removed R18, R20, R22, R6: 10k, Resistor_SMD:R_0402_1005Metric, symbol Device:R_Small
- removed R3: 0R, Resistor_SMD:R_0402_1005Metric, symbol Device:R_Small
- removed R8: 330R, Resistor_SMD:R_0402_1005Metric, symbol Device:R_Small
- removed U5: 74LVC2T45DC, Package_SO:VSSOP-8_2.3x2mm_P0.5mm, symbol Logic_LevelTranslator:74LVC2T45DC
- added NT1: NetTie_2, NetTie:NetTie-2_SMD_Pad0.5mm, symbol Device:NetTie_2
- added Q1, Q2: CJE3139K, Package_TO_SOT_SMD:SOT-523, symbol Debug_Probe_FET:CJE3139K
- added Q5, Q6: 2N7002, Package_TO_SOT_SMD:SOT-523, symbol Transistor_FET:2N7002
- added RN3: 10k, Resistor_SMD:R_Array_Convex_4x0402, symbol Device:R_Pack04_Split
- added TP10, TP11, TP12, TP5, TP6, TP7, TP8, TP9: TestPoint, TestPoint:TestPoint_Pad_D1.5mm, symbol Connector:TestPoint
- C11: LCSC (none) -> C307331
- C14: LCSC (none) -> C15849
- RN1, RN2: value 100R -> 121R; footprint (none) -> Resistor_SMD:R_Array_Convex_4x0402; LCSC (none) -> C728706
- SW1: LCSC (none) -> C262416; lcsc C262416 -> (none)
- U1: LCSC (none) -> C5180249; lcsc C5180249 -> (none)
Connections:
- net +3V3: now also NT1.1, Q1.3, TP10.1; no longer C11.1, C12.1, U3.9 (VDDA)
- net GND: now also Q5.2 (S), Q6.2 (S), RN3.1 (R1.1), RN3.7 (R2.2), TP9.1
- net PWR_BR: now also Q1.1, Q2.1, RN3.5 (R4.2)
- net RST_SENSE: now also Q6.3 (D)
- net SWCLK: now also TP6.1
- net SWDIO: now also TP7.1
- net SWO: now also TP8.1
- net TCK: now also RN1.3 (R3.1); no longer RN1.2 (R2.1)
- net TDI: now also RN1.1 (R1.1); no longer RN1.4 (R4.1)
- net TDO: now also RN1.2 (R2.1); no longer RN1.3 (R3.1)
- net TMS: now also RN1.4 (R4.1); no longer RN1.1 (R1.1)
- net TPWR: now also Q2.3
- net TPWR_MEAS: now also RN3.2 (R2.1)
- net VBUS_MEAS: now also RN3.8 (R1.2)
- net iRST: now also Q5.1 (G)
- net iRXD: now also TP12.1; no longer U7.3 (2A)
- net iTXD: now also TP11.1
- net nRST: now also C9.1, U3.7 (NRST), TP5.1
- net xRST: now also RN2.8 (R1.2), Q5.3 (D), Q6.1 (G), RN3.6 (R3.2)
- net xTCK: now also RN1.6 (R3.2); no longer RN1.7 (R2.2)
- net xTDI: now also RN1.8 (R1.2); no longer RN1.5 (R4.2)
- net xTDO: now also RN1.7 (R2.2); no longer RN1.6 (R3.2)
- net xTMS: now also RN1.5 (R4.2); no longer RN1.8 (R1.2)
- net xTPWR: now also RN3.3 (R3.1)
- net LED0: no longer names the net of U3.20 (PB2)
- net RXD: no longer names the net of RN2.3 (R3.1)
- net TXD: no longer names the net of RN2.2 (R2.1)
- net xRXD: no longer names the net of RN2.6 (R3.2)
- net xRXD: no longer U7.6 (2B)
- net xTXD: no longer names the net of RN2.7 (R2.2)
- new net: Q1.2, Q2.2, RN3.4 (R4.1)
- new net VDDA: C11.1, C12.1, NT1.2, U3.9 (VDDA)
- no-connect marks 26 -> 31
Other:
- note added: "LED0 excluded for space constraint"
- note added: "Programming/Debug Header"
- note removed: "-> <-"
- note removed: "Tag Connect"
- note removed: "UART header mounted sideways sticking off edge of board"
- moved on the sheet: C6, RN1A, RN1B, RN1C, RN1D, U6, U7, U8

Commit message: part numbers
Parts:
- R1, R2: LCSC (none) -> C881131
- R10, R9: LCSC (none) -> C25104
- R21, R5: LCSC (none) -> C163826
- R4: value 10k -> 220k; LCSC (none) -> C25767
- U6, U8: LCSC (none) -> C2652936
Other:
- moved on the sheet: D2, D3, J2, R10, RN1A, RN1B, RN1C, RN1D, RN2A, RN2B, RN2C, TP10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

Commit message: update part numbers
Parts:
- C11, C14, C3: LCSC C15849 -> C52923
- U3: LCSC C77994 -> C8734
Changed lines of the file:
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@@
       (effects (font (size 1.27 1.27)) hide)
     )
-    (property "LCSC" "C15849" (at 107.95 45.72 0)
+    (property "LCSC" "C52923" (at 107.95 45.72 0)
       (effects (font (size 1.27 1.27)) hide)
     )
@@
       (effects (font (size 1.27 1.27)) hide)
     )
-    (property "LCSC" "C15849" (at 135.89 45.72 0)
+    (property "LCSC" "C52923" (at 135.89 45.72 0)
       (effects (font (size 1.27 1.27)) hide)
     )
@@
       (effects (font (size 1.27 1.27)) hide)
     )
-    (property "LCSC" "C15849" (at 90.17 146.05 0)
+    (property "LCSC" "C52923" (at 90.17 146.05 0)
       (effects (font (size 1.27 1.27)) hide)
     )
@@
       (effects (font (size 1.27 1.27)) hide)
     )
-    (property "LCSC" "C77994" (at 99.06 210.82 0)
-      (effects (font (size 1.27 1.27)) hide)
-    )
+    (property "LCSC" "C8734" (at 99.06 210.82 0)
+      (effects (font (size 1.27 1.27)) hide)
+    )

Commit message: made usb2can schematic/pcb
Parts:
- removed C12 (x2), C6 (x6), C9: 100n, Capacitor_SMD:C_0402_1005Metric, symbol Device:C_Small
- removed C5, C7: 30p, Capacitor_SMD:C_0402_1005Metric, symbol Device:C_Small
- removed J2: Conn_ARM_JTAG_SWD_10, Connectors:Cortex-10pin-sidemount, symbol Connector:Conn_ARM_JTAG_SWD_10
- removed Q1, Q2: CJE3139K, Package_TO_SOT_SMD:SOT-523, symbol Debug_Probe_FET:CJE3139K
- removed Q5, Q6: 2N7002, Package_TO_SOT_SMD:SOT-523, symbol Transistor_FET:2N7002
- removed R21: 4k7, Resistor_SMD:R_0402_1005Metric, symbol Device:R_Small
- removed R6: 1k5, Resistor_SMD:R_0402_1005Metric, symbol Device:R_Small
- removed RN1, RN2: 121R, Resistor_SMD:R_Array_Convex_4x0402, symbol Device:R_Pack04_Split
- removed RN3: 10k, Resistor_SMD:R_Array_Convex_4x0402, symbol Device:R_Pack04_Split
- removed TP10, TP11, TP12, TP5, TP6, TP7, TP8, TP9: TestPoint, TestPoint:TestPoint_Pad_D1.5mm, symbol Connector:TestPoint
- removed U3: STM32F103C8T6, Package_QFP:LQFP-48_7x7mm_P0.5mm, symbol MCU_ST_STM32F1:STM32F103C8Tx
- removed U6, U7, U8: 74LVC2T45DC, Package_SO:VSSOP-8_2.3x2mm_P0.5mm, symbol Logic_LevelTranslator:74LVC2T45DC
- removed Y1: 8MHz, Crystal:Crystal_SMD_5032-2Pin_5.0x3.2mm, symbol Device:Crystal_Small
- added C10 (x2): 100n, Capacitor_SMD:C_0402_1005Metric, symbol Device:C_Small
- added J1: TC2030-NL, Connector:Tag-Connect_TC2030-IDC-NL_2x03_P1.27mm_Vertical, symbol Connector:Conn_ARM_SWD_TagConnect_TC2030-NL
- added J2: Conn_01x04, Connectors:p3_5_edge_header, symbol Connector_Generic:Conn_01x04
- added JP1: TERM, Jumper:SolderJumper-2_P1.3mm_Open_TrianglePad1.0x1.5mm, symbol Jumper:SolderJumper_2_Open
- added JP2: RESET, Jumper:SolderJumper-2_P1.3mm_Open_TrianglePad1.0x1.5mm, symbol Jumper:SolderJumper_2_Open
- added R3: 220k, Resistor_SMD:R_0402_1005Metric, symbol Device:R_Small
- added U2: TCAN1042HGVDQ1, tcan1042:D0008A_N, symbol TCAN1042:TCAN1042HGVDQ1
- added U3: STM32G431CBUx, Package_DFN_QFN:QFN-48-1EP_7x7mm_P0.5mm_EP5.6x5.6mm, symbol MCU_ST_STM32G4:STM32G431CBUx
- D2: value Orange -> Blue
- D3: value Red -> Green
- R4: value 220k -> 120; footprint Resistor_SMD:R_0402_1005Metric -> Resistor_SMD:R_1206_3216Metric; LCSC C25767 -> C17909
- R5: value 4k7 -> 330R; LCSC C163826 -> C25104
- SW1: value SW_Push -> BOOT
Connections:
- net +3V3: now also SW1.1, J1.1 (VCC), U3.1 (VBAT), U3.23 (VDD), U3.35 (VDD), U3.48 (VDD); no longer R4.2
- net GND: now also C10.2, C10.2, J1.5 (GND), J2.1 (Pin_1), R3.2, U2.2 (GND), U3.49 (VSS); no longer SW1.1
- net SWCLK: now also J1.4 (SWCLK), U3.37 (PA14)
- net SWDIO: now also J1.2 (SWDIO), U3.36 (PA13)
- net SWO: now also J1.6 (SWO), U3.41 (PB3)
- net USB_D+: now also U3.34 (PA12)
- net USB_D-: now also U3.33 (PA11)
- net VBUS: now also C10.1, J2.4 (Pin_4), U2.3 (VCC); no longer R5.2
- net VDDA: now also U3.20 (VREF+), U3.21 (VDDA)
- net at R4.1: now also J2.3 (Pin_3), U2.7 (CANH); no longer SW1.2
- net LED1 renamed LEDB
- net LEDB: now also U3.38 (PA15)
- net LED2 renamed LEDG
- net LEDG: now also U3.24 (PB11)
- net VBUS_MEAS: no longer names the net of R5.1
- net VBUS_MEAS: now also JP2.1 (A)
- new net: R5.2, U3.7 (PG10)
- new net: JP1.2 (B), R4.2
- new net: J2.2 (Pin_2), JP1.1 (A), U2.6 (CANL)
- new net CANRX: R3.1, SW1.2, U2.4 (RXD), U3.46 (PB8)
- new net CANTX: U2.1 (TXD), U3.47 (PB9)
- new net CAN_IOPWR: C10.1, U2.5 (VIO), U3.2 (PC13)
- new net CAN_STBY: U2.8 (STB), U3.8 (PA0)
- new net nRESET: J1.3 (~{RESET}), JP2.2 (B)
- no-connect marks 31 -> 40
Other:
- note added: "CAN Transceiver"
- note added: "STM32G431 Microcontroller"
- note removed: "CL = 2 * (Cload - Cstray)"
- note removed: "JTAG header mounted on side of board with 1/2 of pins on top and 1/2 on bottom"
- note removed: "LED0 excluded for space constraint"
- note removed: "Level conversion & Target Frontend"
- note removed: "STM32F1 Microcontroller"
- note removed: "STM32F103 requires external 1k5 pull-up on USB D+ line."
- moved on the sheet: D2, D3, R10
