File: pcb.kicad_pcb (KiCad board)
At the start: 4 copper layers, 26 x 30 mm, 71 parts, among them J1 Conn_ARM_SWD_TagConnect_TC203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, J2 Conn_ARM_JTAG_SWD_10, J3 JST B04B-PASK, P1 USB_C_Plug, Q1 AO3400A, Q2 AO3400A, Q3 AO3401A, Q4 AO3401A, SW1 SW_Push, U1 WE-TVS-82400102, U2 STM32F103C8T6, U5 74LVC2T45DC, U6 74LVC2T45DC, U7 74LVC2T45DC, U8 74LVC2T45DC, U9 AP2112K-3.3, Y1 8MHz

Commit message: Layout and routing
Parts:
- removed C16, C20: 100n, Capacitor_SMD:C_0402_1005Metric
- removed D1: Yellow, Connectors:LED_THT_Edge Mount
- removed J1: Conn_ARM_SWD_TagConnect_TC2030-NL, Connector:Tag-Connect_TC2030-IDC-NL_2x03_P1.27mm_Vertical
- removed J3: JST B04B-PASK, Connectors:JST B04B-PASK Edge Mount
- removed Q3, Q4: AO3401A, Package_TO_SOT_SMD:SOT-23
- removed R11, R12, R13, R14, R15, R16, R17, R19: 100R, Resistor_SMD:R_0402_1005Metric
- removed R18, R20, R22, R6: 10k, Resistor_SMD:R_0402_1005Metric
- removed R3: 0R, Resistor_SMD:R_0402_1005Metric
- removed R8: 330R, Resistor_SMD:R_0402_1005Metric
- removed U5: 74LVC2T45DC, Package_SO:VSSOP-8_2.3x2mm_P0.5mm
- added G***: LOGO, framework-debug-probe:pretzel, B.Cu at (132.4, 86.5)
- added NT1: NetTie_2, NetTie:NetTie-2_SMD_Pad0.5mm, F.Cu at (133.9, 84.5)
- added Q5: 2N7002, Package_TO_SOT_SMD:SOT-523, F.Cu at (150.9, 80.1)
- added Q6: 2N7002, Package_TO_SOT_SMD:SOT-523, F.Cu at (150.9, 82.3)
- added RN1: 121R, Resistor_SMD:R_Array_Convex_4x0402, F.Cu at (137.0, 94.0)
- added RN2: 121R, Resistor_SMD:R_Array_Convex_4x0402, F.Cu at (146.5, 94.0)
- added RN3: 10k, Resistor_SMD:R_Array_Convex_4x0402, F.Cu at (148.6, 80.0)
- added TP10: TestPoint, TestPoint:TestPoint_Pad_D1.5mm, B.Cu at (151.3, 86.1)
- added TP11: TestPoint, TestPoint:TestPoint_Pad_D1.5mm, B.Cu at (142.0, 82.7)
- added TP12: TestPoint, TestPoint:TestPoint_Pad_D1.5mm, B.Cu at (142.0, 79.2)
- added TP5: TestPoint, TestPoint:TestPoint_Pad_D1.5mm, B.Cu at (151.3, 73.4)
- added TP6: TestPoint, TestPoint:TestPoint_Pad_D1.5mm, B.Cu at (151.3, 78.5)
- added TP7: TestPoint, TestPoint:TestPoint_Pad_D1.5mm, B.Cu at (151.3, 81.0)
- added TP8: TestPoint, TestPoint:TestPoint_Pad_D1.5mm, B.Cu at (151.3, 75.9)
- added TP9: TestPoint, TestPoint:TestPoint_Pad_D1.5mm, B.Cu at (151.3, 83.6)
- Q1, Q2: value AO3400A -> CJE3139K; footprint Package_TO_SOT_SMD:SOT-23 -> Package_TO_SOT_SMD:SOT-523
- moved D3 18.0 mm to (131.8, 95.1)
- moved R10 15.3 mm to (133.4, 94.7), turned to -90 degrees
- moved C24 14.1 mm to (147.1, 79.5), turned to 90 degrees
- moved C7 13.6 mm to (152.8, 73.5), turned to -90 degrees
- moved R21 13.5 mm to (147.0, 82.5), turned to -90 degrees
- moved C18 13.0 mm to (145.7, 88.2)
- moved C22 13.0 mm to (145.7, 90.8)
- moved U7 12.9 mm to (143.8, 89.5)
- moved Q2 12.4 mm to (148.5, 82.5), turned to -90 degrees
- moved C13 10.7 mm to (151.3, 73.2), turned to 180 degrees
- moved R4 10.5 mm to (151.3, 75.2)
- moved R5 8.48 mm to (151.3, 74.2), turned to 180 degrees
- moved Q1 8.12 mm to (148.5, 85.1)
- moved D2 7.27 mm to (151.8, 95.1)
- moved C19 7.18 mm to (138.1, 88.3)
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Connections:
- C10 pad 1: +3V3 -> VDDA
- C7 pad 1: Net-(U2-NRST) -> nRST
- C9 pad 1: +3V3 -> VDDA
- Q1 pad 1: iRST -> PWR_BR
- Q1 pad 2: GND -> Net-(RN3D-R4.1)
- Q1 pad 3: xRST -> +3V3
- Q2 pad 1: xRST -> PWR_BR
- Q2 pad 2: GND -> Net-(RN3D-R4.1)
- Q2 pad 3: RST_SENSE -> TPWR
- U2 pad 20: LED0 -> unconnected-(U2-PB2-Pad20)
- U2 pad 7: Net-(U2-NRST) -> nRST
- U2 pad 9: +3V3 -> VDDA
- U7 pad 3: iRXD -> unconnected-(U7-2A-Pad3)
- U7 pad 6: xRXD -> unconnected-(U7-2B-Pad6)
Routing:
- net GND: track 0.00 -> 78.6 mm, vias 8 -> 52
- net +3V3: track 0.00 -> 30.9 mm, vias 0 -> 20
- net nRST: track 0.00 -> 21.8 mm, vias 0 -> 2
- net iRST: track 0.00 -> 21.8 mm, vias 0 -> 2
- net xTPWR: track 0.00 -> 19.7 mm, vias 0 -> 6
- net Net-(U2-PB12): track 0.00 -> 18.6 mm, vias 0 -> 2
- net VBUS_MEAS: track 0.00 -> 18.6 mm, vias 0 -> 2
- net LED1: track 0.00 -> 18.2 mm, vias 0 -> 2
- net LED2: track 0.00 -> 17.8 mm, vias 0 -> 2
- net RST_SENSE: track 0.00 -> 17.6 mm, vias 0 -> 2
- net TPWR: track 0.00 -> 17.0 mm
- net xRST: track 0.00 -> 16.9 mm
- net PWR_BR: track 0.00 -> 16.0 mm, vias 0 -> 2
- net iTDO: track 0.00 -> 15.7 mm
- net VBUS: track 0.00 -> 15.2 mm, vias 0 -> 8
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- added copper zone on In2.Cu, net +3V3
- added copper zone on B.Cu, net GND
- added copper zone on In1.Cu, net GND
- added copper zone on F.Cu, net VBUS
- added copper zone on In2.Cu, net VBUS
- added copper zone on In2.Cu, net xTPWR
Other:
- board size 26 x 30 mm -> 26 x 25.6 mm
- board text added: "3V3"
- board text added: "BOOT"
- board text added: "ERROR"
- board text added: "Framework Debug Probe"
- board text added: "GND"
- board text added: "IDLE"
- board text added: "JTAG SWD"
- board text added: "Jack LeFevre"
- board text added: "RST"
- board text added: "RXD"
- board text added: "SWCLK"
- board text added: "SWDIO"
- board text added: "SWO"
- board text added: "TMS SWDIO TCK SWCLK TDO SWO TDI ~{RESET}"
- board text added: "TXD"
- board text added: "rev 0.1 June 2023"

Commit message: part numbers
Parts:
- R4: value 10k -> 220k
Changed lines of the file:
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@@
     (descr "Resistor SMD 0402 (1005 Metric), square (rectangular) end terminal, IPC_7351 nominal, (Body size source: IPC-SM-782 page 72, https://www.pcb-3d.com/wordpress/wp-content/uploads/ipc-sm-782a_amendment_1_and_2.pdf), generated with kicad-footprint-generator")
     (tags "resistor")
+    (property "LCSC" "C25104")
     (property "Sheetfile" "pcb.kicad_sch")
     (property "Sheetname" "")
@@
     (descr "Resistor SMD 0402 (1005 Metric), square (rectangular) end terminal, IPC_7351 nominal, (Body size source: IPC-SM-782 page 72, https://www.pcb-3d.com/wordpress/wp-content/uploads/ipc-sm-782a_amendment_1_and_2.pdf), generated with kicad-footprint-generator")
     (tags "resistor")
+    (property "LCSC" "C163826")
     (property "Sheetfile" "pcb.kicad_sch")
     (property "Sheetname" "")
@@
     (descr "Resistor SMD 0402 (1005 Metric), square (rectangular) end terminal, IPC_7351 nominal, (Body size source: IPC-SM-782 page 72, https://www.pcb-3d.com/wordpress/wp-content/uploads/ipc-sm-782a_amendment_1_and_2.pdf), generated with kicad-footprint-generator")
     (tags "resistor")
+    (property "LCSC" "C25767")
     (property "Sheetfile" "pcb.kicad_sch")
     (property "Sheetname" "")
@@
         (effects (font (size 1 1) (thickness 0.15)))
     )
-    (fp_text value "10k" (at 0 1.17) (layer "F.Fab")
+    (fp_text value "220k" (at 0 1.17) (layer "F.Fab")
         (effects (font (size 1 1) (thickness 0.15)))
     )
@@
     (descr "Resistor SMD 0402 (1005 Metric), square (rectangular) end terminal, IPC_7351 nominal, (Body size source: IPC-SM-782 page 72, https://www.pcb-3d.com/wordpress/wp-content/uploads/ipc-sm-782a_amendment_1_and_2.pdf), generated with kicad-footprint-generator")
     (tags "resistor")
+    (property "LCSC" "C881131")
     (property "Sheetfile" "pcb.kicad_sch")
     (property "Sheetname" "")
@@
     (descr "VSSOP-8 2.3x2mm Pitch 0.5mm")
     (tags "VSSOP-8 2.3x2mm Pitch 0.5mm")
+    (property "LCSC" "C2652936")
     (property "Sheetfile" "pcb.kicad_sch")
     (property "Sheetname" "")
@@
     (descr "Resistor SMD 0402 (1005 Metric), square (rectangular) end terminal, IPC_7351 nominal, (Body size source: IPC-SM-782 page 72, https://www.pcb-3d.com/wordpress/wp-content/uploads/ipc-sm-782a_amendment_1_and_2.pdf), generated with kicad-footprint-generator")
     (tags "resistor")
+    (property "LCSC" "C163826")
     (property "Sheetfile" "pcb.kicad_sch")
     (property "Sheetname" "")
@@
     (descr "Resistor SMD 0402 (1005 Metric), square (rectangular) end terminal, IPC_7351 nominal, (Body size source: IPC-SM-782 page 72, https://www.pcb-3d.com/wordpress/wp-content/uploads/ipc-sm-782a_amendment_1_and_2.pdf), generated with kicad-footprint-generator")
     (tags "resistor")
+    (property "LCSC" "C25104")
     (property "Sheetfile" "pcb.kicad_sch")
     (property "Sheetname" "")
@@
     (descr "Resistor SMD 0402 (1005 Metric), square (rectangular) end terminal, IPC_7351 nominal, (Body size source: IPC-SM-782 page 72, https://www.pcb-3d.com/wordpress/wp-content/uploads/ipc-sm-782a_amendment_1_and_2.pdf), generated with kicad-footprint-generator")
     (tags "resistor")
+    (property "LCSC" "C881131")
     (property "Sheetfile" "pcb.kicad_sch")
     (property "Sheetname" "")
@@
     (descr "VSSOP-8 2.3x2mm Pitch 0.5mm")
     (tags "VSSOP-8 2.3x2mm Pitch 0.5mm")
-    (property "Sheetfile" "pcb.kicad_sch")
-    (property "Sheetname" "")
+    (property "LCSC" "C2652936")
+    (property "Sheetfile" "pcb.kicad_sch")
+    (property "Sheetname" "")

Commit message: move parts around
Parts:
- G***: footprint framework-debug-probe:pretzel -> Connectors:pretzel
Changed lines of the file:
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@@
       (net 17 "SWO") (pinfunction "1") (pintype "passive"))
   )
-  (footprint "framework-debug-probe:pretzel" (layer "B.Cu")
+  (footprint "Connectors:pretzel" (layer "B.Cu")
     (at 132.42 86.5 90)
     (attr board_only exclude_from_pos_files exclude_from_bom)
-    (fp_text reference "G***" (at 0 0 90) (layer "B.SilkS") hide
+    (fp_text reference "G***" (at 0 0 270) (layer "B.SilkS") hide
         (effects (font (size 1.5 1.5) (thickness 0.3)) (justify mirror))
     )
-    (fp_text value "LOGO" (at 0.75 0 90) (layer "B.SilkS") hide
+    (fp_text value "LOGO" (at 0.75 0 270) (layer "B.SilkS") hide
         (effects (font (size 1.5 1.5) (thickness 0.3)) (justify mirror))
     )

Commit message: made usb2can schematic/pcb
Parts:
- removed C13, C17, C18, C19, C21, C22, C23, C24, C7: 100n, Capacitor_SMD:C_0402_1005Metric
- removed Q1, Q2: CJE3139K, Package_TO_SOT_SMD:SOT-523
- removed Q5, Q6: 2N7002, Package_TO_SOT_SMD:SOT-523
- removed R21: 4k7, Resistor_SMD:R_0402_1005Metric
- removed R7: 1k5, Resistor_SMD:R_0402_1005Metric
- removed RN1, RN2: 121R, Resistor_SMD:R_Array_Convex_4x0402
- removed RN3: 10k, Resistor_SMD:R_Array_Convex_4x0402
- removed TP10, TP11, TP12, TP5, TP6, TP7, TP8, TP9: TestPoint, TestPoint:TestPoint_Pad_D1.5mm
- removed U6, U7, U8: 74LVC2T45DC, Package_SO:VSSOP-8_2.3x2mm_P0.5mm
- removed Y1: 8MHz, Crystal:Crystal_SMD_5032-2Pin_5.0x3.2mm
- added J1: TC2030-NL, Connector:Tag-Connect_TC2030-IDC-NL_2x03_P1.27mm_Vertical, B.Cu at (139.7, 78.3)
- added JP1: TERM, Jumper:SolderJumper-2_P1.3mm_Open_TrianglePad1.0x1.5mm, B.Cu at (134.5, 85.8)
- added JP2: RESET, Jumper:SolderJumper-2_P1.3mm_Open_TrianglePad1.0x1.5mm, B.Cu at (134.5, 81.8)
- added R3: 220k, Resistor_SMD:R_0402_1005Metric, F.Cu at (142.7, 83.9)
- added U3: STM32G431CBUx, Package_DFN_QFN:QFN-48-1EP_7x7mm_P0.5mm_EP5.6x5.6mm, F.Cu at (147.4, 82.9)
- C1, C2: value 30p -> 100n
- D2: value Orange -> Blue
- D3: value Red -> Green
- J2: value Conn_ARM_JTAG_SWD_10 -> Conn_01x04; footprint Connectors:Cortex-10pin-sidemount -> Connectors:p3_5_edge_header; moved to B.Cu
- R4: value 220k -> 120; footprint Resistor_SMD:R_0402_1005Metric -> Resistor_SMD:R_1206_3216Metric
- R5: value 4k7 -> 330R
- SW1: value SW_Push -> BOOT
- U2: value STM32F103C8T6 -> TCAN1042HGVDQ1; footprint Package_QFP:LQFP-48_7x7mm_P0.5mm -> tcan1042:D0008A_N
- moved R4 21.3 mm to (135.4, 89.3)
- moved C9 19.8 mm to (153.2, 82.9), turned to -90 degrees
- moved NT1 19.5 mm to (153.1, 80.9), turned to -90 degrees
- moved C10 17.6 mm to (152.1, 82.9), turned to -90 degrees
- moved G*** 15.6 mm to (147.3, 81.8)
- moved R5 14.1 mm to (147.1, 87.6), turned to 0 degrees
- moved C5 14.0 mm to (144.2, 87.6), turned to 180 degrees
- moved C8 12.0 mm to (142.7, 86.4), turned to -90 degrees
- moved C6 8.96 mm to (152.1, 80.0)
- moved SW1 7.32 mm to (141.1, 83.0), turned to 0 degrees
- moved U2 6.81 mm to (134.2, 84.0), turned to -90 degrees
- moved C1 6.74 mm to (130.9, 86.2), turned to 90 degrees
- moved J2 3.52 mm to (141.9, 90.7), turned to 0 degrees
- moved C2 1.30 mm to (134.3, 79.6), turned to 0 degrees
- moved C4 0.56 mm to (144.8, 77.7), turned to 90 degrees
Connections:
- net /HSE_OUT renamed CAN_IOPWR
- C2 pad 1: /HSE_IN -> VBUS
- J2 pad 1: TPWR -> GND
- J2 pad 2: /TMS -> Net-(J2-Pin_2)
- J2 pad 3: GND -> Net-(J2-Pin_3)
- J2 pad 4: /TCK -> VBUS
- R10 pad 1: LED2 -> LEDG
- R4 pad 1: Net-(U2-PB12) -> Net-(J2-Pin_3)
- R4 pad 2: +3V3 -> Net-(JP1-B)
- R5 pad 1: VBUS_MEAS -> Net-(JP2-A)
- R5 pad 2: VBUS -> Net-(U3-PG10)
- R9 pad 1: LED1 -> LEDB
- SW1 pad 1: GND -> +3V3
- SW1 pad 2: Net-(U2-PB12) -> CANRX
- U2 pad 1: +3V3 -> CANTX
- U2 pad 2: unconnected-(U2-PC13-Pad2) -> GND
- U2 pad 3: unconnected-(U2-PC14-Pad3) -> VBUS
- U2 pad 4: unconnected-(U2-PC15-Pad4) -> CANRX
- U2 pad 6: /HSE_IN -> Net-(J2-Pin_2)
- U2 pad 7: nRST -> Net-(J2-Pin_3)
- U2 pad 8: GND -> CAN_STBY
Routing:
- net GND: track 78.6 -> 33.3 mm, vias 52 -> 34
- net LEDG: track 0.00 -> 36.7 mm
- net nRST: track 21.8 -> 0.00 mm, vias 2 -> 0
- net iRST: track 21.8 -> 0.00 mm, vias 2 -> 0
- net LEDB: track 0.00 -> 19.9 mm, vias 0 -> 2
- net xTPWR: track 19.7 -> 0.00 mm, vias 6 -> 0
- net Net-(U2-PB12): track 18.6 -> 0.00 mm, vias 2 -> 0
- net VBUS_MEAS: track 18.6 -> 0.00 mm, vias 2 -> 0
- net CANRX: track 0.00 -> 18.5 mm, vias 0 -> 1
- net LED1: track 18.2 -> 0.00 mm, vias 2 -> 0
- net LED2: track 17.8 -> 0.00 mm, vias 2 -> 0
- net VBUS: track 15.2 -> 33.0 mm
- net RST_SENSE: track 17.6 -> 0.00 mm, vias 2 -> 0
- net TPWR: track 17.0 -> 0.00 mm
- net xRST: track 16.9 -> 0.00 mm
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- removed copper zone on In2.Cu, net xTPWR
Other:
- outline, holes or cut-outs redrawn
- board text added: "BLUE"
- board text added: "Framework USB2CAN"
- board text added: "GREEN"
- board text added: "rev 0.1 Sept 2023"
- board text removed: "3V3"
- board text removed: "ERROR"
- board text removed: "Framework Debug Probe"
- board text removed: "GND"
- board text removed: "IDLE"
- board text removed: "JTAG SWD"
- board text removed: "RST"
- board text removed: "RXD"
- board text removed: "SWCLK"
- board text removed: "SWDIO"
- board text removed: "SWO"
- board text removed: "TMS SWDIO TCK SWCLK TDO SWO TDI ~{RESET}"
- board text removed: "TXD"
- board text removed: "rev 0.1 June 2023"
